Commit message: added the include xacro file

File: description/robot.urdf.xacro (robot description, xacro)
@@ -1,4 +1,4 @@
 <?xml version="1.0"?>
 <robot xmlns:xacro="http://www.ros.org/wiki/xacro"  name="robot">
-    <link name="base_link"></link>
+    <xacro:include filename = "robot_core.xacro"/>
 </robot>
