Commit message: xacro file modified

File: description/robot_core.xacro (robot description, xacro)
@@ -1,3 +1,65 @@
 <?xml version="1.0"?>
 <robot xmlns:xacro="http://www.ros.org/wiki/xacro">
+    <!-- material properties : color-->
+    <material name = "white">
+        <color rgba = "1 1 1 1"/>
+    </material>
+    <material name = "orange">
+        <color rgba = "1 0.3 0.001 1"/>
+    </material>
+    <material name = "blue">
+        <color rgba = "0.2 0.2 1 1"/>
+    </material>
+    <material name = "black">
+        <color rgba = "0.025 0.025 0.025 1"/>
+    </material>
+    <!-- robot links-->
+    <!-- base Link-->
+    <link name = "base_link">
+    </link>
+    <!-- Chassis Link-->
+    <joint name = "chassis_joint" type = "fixed">
+        <parent link = "base_link"/>
+        <child link = "chassis"/>
+        <origin xyz = "-0.1 0 0"/>
+    </joint>
+    <link name = "chassis">
+        <visual>
+            <origin xyz = "0.15 0 0.075"/>
+            <geometry>
+                <box size = "0.3 0.3 0.15"/>
+            </geometry>
+            <material name = "white"/>
+        </visual>
+    </link>
+    <!-- Left Wheel-->
+    <joint name = "left_wheel_joint" type ="continuous">
+        <parent link = "base_link"/>
+        <child link = "left_wheel"/>
+        <origin xyz = "0 0.175 0" rpy = "-${pi/2} 0 0"/>
+        <axis xyz = "0 0 1"/>
+    </joint>
+    <link name = "left_wheel">
+        <visual>
+            <geometry>
+                <cylinder radius = "0.05" length = "0.04"/>
+            </geometry>
+            <material name = "black"/>
+        </visual>
+    </link>
+    <!-- Right Wheel-->
+    <joint name = "right_wheel_joint" type ="continuous">
+        <parent link = "base_link"/>
+        <child link = "right_wheel"/>
+        <origin xyz = "0 -0.175 0" rpy = "${pi/2} 0 0"/>
+        <axis xyz = "0 0 1"/>
+    </joint>
+    <link name = "left_wheel">
+        <visual>
+            <geometry>
+                <cylinder radius = "0.05" length = "0.04"/>
+            </geometry>
+            <material name = "black"/>
+        </visual>
+    </link>
 </robot>
